Commit message: More precise inertia and mass data

File: urdf/robot_simplified.urdf (robot description, URDF)
Before this commit: robot robot, 6 links, 5 joints
Links:
- link LF_CALF: mass 1.634976467 -> 0.082921
- link LF_FOOT: mass 0.207204302 -> 0.0023701
- link LF_THIGH: mass 1.42462064 -> 0.497881
- link base_inertia: mass 16.793507758 -> 0.2565404

Commit message: Adding revolute joint as a z constraint

File: urdf/robot_simplified.urdf (robot description, URDF)
Before this commit: robot robot, 6 links, 5 joints
Links:
- removed link base_inertia
- added link base_inertial, mass 0.2565404; collision box size=0.4 0.2 0.05; visual box size=0.4 0.2 0.05
- link base: geometry visual sphere radius=0.02
Joints:
- removed joint base_to_base_inertia
- added joint base_to_base_inertial: type prismatic, parent base, child base_inertial, origin xyz=0 0 0 rpy=0 0 0, axis 0 0 1, limit lower=-10 upper=30 effort=1000.0 velocity=10
- joint LF_JHIP: parent base -> base_inertial

Commit message: Remove prismatic joint - handle it in control software

File: urdf/robot_simplified.urdf (robot description, URDF)
Before this commit: robot robot, 6 links, 5 joints
Joints:
- joint base_to_base_inertial: type prismatic -> fixed

Commit message: Better torque and position limits

File: urdf/robot_simplified.urdf (robot description, URDF)
Before this commit: robot robot, 6 links, 5 joints
Joints:
- joint LF_JANCKLE: limit lower=-9.42 upper=9.42 effort=80 velocity=15.0 -> lower=-10.0 upper=10.0 effort=6.0 velocity=8.0
- joint LF_JHIP: limit lower=-9.42 upper=9.42 effort=80 velocity=15 -> lower=-7.0 upper=7.0 effort=8.0 velocity=6.0
- joint LF_JKNEE: limit lower=-9.42 upper=9.42 effort=80 velocity=15.0 -> lower=-2.0 upper=2.0 effort=7.5 velocity=7.0
